File: pcb/v1/ain.kicad_sch (KiCad schematic)
At the start: 69 parts, among them J1 R_Small, J10 R_Small, J11 R_Small, J12 R_Small, J13 R_Small, J14 R_Small, J15 R_Small, J16 R_Small, J2 R_Small, J3 R_Small, J4 R_Small, J5 R_Small, J6 R_Small, J7 R_Small, J8 R_Small, J9 R_Small, U1 MCP602, U2 MCP602, U4 MCP602

Commit message: Prepared for PCB ordering
Parts:
- added J18, J19, J20: R_Small, Resistor_SMD:R_1206_3216Metric_Pad1.30x1.75mm_HandSolder, symbol Device:R_Small
- renumbered CONN_AIN1 to C_AIN1, CONN_AIN2 to C_AIN2, CONN_AIN3 to C_AIN3, CONN_AIN4 to C_AIN4, CONN_AIN5 to C_AIN5, CONN_AIN6 to C_AIN6
Connections:
- net A3V: now also J18.2, J19.2, J20.2; no longer C1.1, C15.1, C16.1, C4.1, C5.1, C6.1, J1.1, J11.1, J12.1, J3.1, J5.1, J6.1, U1.8 (V+), U2.8 (V+), U4.8 (V+)
- new net: C5.1, C6.1, J19.1, J5.1, J6.1, U2.8 (V+)
- new net: C15.1, C16.1, J11.1, J12.1, J20.1, U4.8 (V+)
- new net: C1.1, C4.1, J1.1, J18.1, J3.1, U1.8 (V+)
