File: pcb/v1/aout.kicad_sch (KiCad schematic)
At the start: 10 parts, among them U3 MCP602

Commit message: Prepared for PCB ordering
Parts:
- renumbered CONN_AOUT1 to C_AOUT1, CONN_AOUT2 to C_AOUT2
Changed lines of the file:
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@@
 		(dnp no)
 		(fields_autoplaced yes)
-		(property "Reference" "CONN_AOUT2"
+		(property "Reference" "C_AOUT2"
 			(at 138.43 87.6299 90)
 			(effects
@@
 			(project "v1"
 				(path "/c9a089ab-5af5-42df-87be-f1df643a1407/61f03f5a-231a-401c-beda-7de2de98f810"
-					(reference "CONN_AOUT2")
+					(reference "C_AOUT2")
 					(unit 1)
 				)
@@
 		(dnp no)
 		(fields_autoplaced yes)
-		(property "Reference" "CONN_AOUT1"
+		(property "Reference" "C_AOUT1"
 			(at 125.73 64.7699 90)
 			(effects
@@
 			(project "v1"
 				(path "/c9a089ab-5af5-42df-87be-f1df643a1407/61f03f5a-231a-401c-beda-7de2de98f810"
-					(reference "CONN_AOUT1")
+					(reference "C_AOUT1")
 					(unit 1)
 				)
