File: pcb/v1/din.kicad_sch (KiCad schematic)
At the start: 42 parts, among them Q1 2N7002K, Q15 2N7002K, Q16 2N7002K, Q2 2N7002K, Q3 2N7002K, Q4 2N7002K

Commit message: Prepared for PCB ordering
Parts:
- renumbered CONN_DIN1 to C_DIN1, CONN_DIN2 to C_DIN2, CONN_DIN3 to C_DIN3, CONN_DIN4 to C_DIN4, CONN_DIN5 to C_DIN5, CONN_DIN6 to C_DIN6
Changed lines of the file:
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@@
 		(dnp no)
 		(fields_autoplaced yes)
-		(property "Reference" "CONN_DIN1"
+		(property "Reference" "C_DIN1"
 			(at 19.558 45.72 90)
 			(effects
@@
 			(project "v1"
 				(path "/c9a089ab-5af5-42df-87be-f1df643a1407/ffc087b2-abba-42aa-b70d-a395e8b765a9"
-					(reference "CONN_DIN1")
+					(reference "C_DIN1")
 					(unit 1)
 				)
@@
 		(dnp no)
 		(fields_autoplaced yes)
-		(property "Reference" "CONN_DIN5"
+		(property "Reference" "C_DIN5"
 			(at 67.818 88.9 90)
 			(effects
@@
 			(project "v1"
 				(path "/c9a089ab-5af5-42df-87be-f1df643a1407/ffc087b2-abba-42aa-b70d-a395e8b765a9"
-					(reference "CONN_DIN5")
+					(reference "C_DIN5")
 					(unit 1)
 				)
@@
 		(dnp no)
 		(fields_autoplaced yes)
-		(property "Reference" "CONN_DIN3"
+		(property "Reference" "C_DIN3"
 			(at 146.558 45.72 90)
 			(effects
@@
 			(project "v1"
 				(path "/c9a089ab-5af5-42df-87be-f1df643a1407/ffc087b2-abba-42aa-b70d-a395e8b765a9"
-					(reference "CONN_DIN3")
+					(reference "C_DIN3")
 					(unit 1)
 				)
@@
 		(dnp no)
 		(fields_autoplaced yes)
-		(property "Reference" "CONN_DIN4"
+		(property "Reference" "C_DIN4"
 			(at 215.138 45.72 90)
 			(effects
@@
 			(project "v1"
 				(path "/c9a089ab-5af5-42df-87be-f1df643a1407/ffc087b2-abba-42aa-b70d-a395e8b765a9"
-					(reference "CONN_DIN4")
+					(reference "C_DIN4")
 					(unit 1)
 				)
@@
 		(dnp no)
 		(fields_autoplaced yes)
-		(property "Reference" "CONN_DIN2"
+		(property "Reference" "C_DIN2"
 			(at 80.518 45.72 90)
 			(effects
@@
 			(project "v1"
 				(path "/c9a089ab-5af5-42df-87be-f1df643a1407/ffc087b2-abba-42aa-b70d-a395e8b765a9"
-					(reference "CONN_DIN2")
+					(reference "C_DIN2")
 					(unit 1)
 				)
@@
 		(dnp no)
 		(fields_autoplaced yes)
-		(property "Reference" "CONN_DIN6"
+		(property "Reference" "C_DIN6"
 			(at 135.128 88.9 90)
 			(effects
@@
 			(project "v1"
 				(path "/c9a089ab-5af5-42df-87be-f1df643a1407/ffc087b2-abba-42aa-b70d-a395e8b765a9"
-					(reference "CONN_DIN6")
-					(unit 1)
-				)
+					(reference "C_DIN6")
+					(unit 1)
+				)
