File: pcb/v1/dout.kicad_sch (KiCad schematic)
At the start: 30 parts, among them Q10 2N7002K, Q5 2N7002K, Q7 2N7002K, Q8 2N7002K, Q9 2N7002K

Commit message: Prepared for PCB ordering
Parts:
- renumbered CONN_DOUT1 to C_DOUT1, CONN_DOUT2 to C_DOUT2, CONN_DOUT3 to C_DOUT3, CONN_DOUT4 to C_DOUT4, CONN_DOUT5 to C_DOUT5
Changed lines of the file:
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@@
 		(on_board yes)
 		(dnp no)
-		(property "Reference" "CONN_DOUT5"
+		(property "Reference" "C_DOUT5"
 			(at 205.232 56.642 90)
 			(effects
@@
 			(project "v1"
 				(path "/c9a089ab-5af5-42df-87be-f1df643a1407/dae6130b-bcb5-41c9-a491-3b23e8945132"
-					(reference "CONN_DOUT5")
+					(reference "C_DOUT5")
 					(unit 1)
 				)
@@
 		(on_board yes)
 		(dnp no)
-		(property "Reference" "CONN_DOUT4"
+		(property "Reference" "C_DOUT4"
 			(at 168.402 56.642 90)
 			(effects
@@
 			(project "v1"
 				(path "/c9a089ab-5af5-42df-87be-f1df643a1407/dae6130b-bcb5-41c9-a491-3b23e8945132"
-					(reference "CONN_DOUT4")
+					(reference "C_DOUT4")
 					(unit 1)
 				)
@@
 		(on_board yes)
 		(dnp no)
-		(property "Reference" "CONN_DOUT3"
+		(property "Reference" "C_DOUT3"
 			(at 130.302 56.642 90)
 			(effects
@@
 			(project "v1"
 				(path "/c9a089ab-5af5-42df-87be-f1df643a1407/dae6130b-bcb5-41c9-a491-3b23e8945132"
-					(reference "CONN_DOUT3")
+					(reference "C_DOUT3")
 					(unit 1)
 				)
@@
 		(on_board yes)
 		(dnp no)
-		(property "Reference" "CONN_DOUT2"
+		(property "Reference" "C_DOUT2"
 			(at 90.932 56.642 90)
 			(effects
@@
 			(project "v1"
 				(path "/c9a089ab-5af5-42df-87be-f1df643a1407/dae6130b-bcb5-41c9-a491-3b23e8945132"
-					(reference "CONN_DOUT2")
+					(reference "C_DOUT2")
 					(unit 1)
 				)
@@
 		(on_board yes)
 		(dnp no)
-		(property "Reference" "CONN_DOUT1"
+		(property "Reference" "C_DOUT1"
 			(at 50.292 56.642 90)
 			(effects
@@
 			(project "v1"
 				(path "/c9a089ab-5af5-42df-87be-f1df643a1407/dae6130b-bcb5-41c9-a491-3b23e8945132"
-					(reference "CONN_DOUT1")
-					(unit 1)
-				)
+					(reference "C_DOUT1")
+					(unit 1)
+				)
