File: pcb/v1/dout_p.kicad_sch (KiCad schematic)
At the start: 22 parts, among them Q12 35N06, Q13 35N06, Q14 2N7002K, Q6 35N06

Commit message: Prepared for PCB ordering
Parts:
- renumbered CONN_DOUT_P1 to C_DOUT_P1, CONN_DOUT_P2 to C_DOUT_P2, CONN_DOUT_P3 to C_DOUT_P3, CONN_DOUT_P_GND1 to C_DOUT_P_GND1
Changed lines of the file:
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@@
 		(dnp no)
 		(fields_autoplaced yes)
-		(property "Reference" "CONN_DOUT_P1"
+		(property "Reference" "C_DOUT_P1"
 			(at 62.23 63.4999 90)
 			(effects
@@
 			(project "v1"
 				(path "/c9a089ab-5af5-42df-87be-f1df643a1407/c1fbf66d-2c5c-4121-915f-86bdae7245e0"
-					(reference "CONN_DOUT_P1")
+					(reference "C_DOUT_P1")
 					(unit 1)
 				)
@@
 		(dnp no)
 		(fields_autoplaced yes)
-		(property "Reference" "CONN_DOUT_P_GND1"
+		(property "Reference" "C_DOUT_P_GND1"
 			(at 63.5 90.1699 90)
 			(effects
@@
 			(project "v1"
 				(path "/c9a089ab-5af5-42df-87be-f1df643a1407/c1fbf66d-2c5c-4121-915f-86bdae7245e0"
-					(reference "CONN_DOUT_P_GND1")
+					(reference "C_DOUT_P_GND1")
 					(unit 1)
 				)
@@
 		(dnp no)
 		(fields_autoplaced yes)
-		(property "Reference" "CONN_DOUT_P3"
+		(property "Reference" "C_DOUT_P3"
 			(at 180.34 63.4999 90)
 			(effects
@@
 			(project "v1"
 				(path "/c9a089ab-5af5-42df-87be-f1df643a1407/c1fbf66d-2c5c-4121-915f-86bdae7245e0"
-					(reference "CONN_DOUT_P3")
+					(reference "C_DOUT_P3")
 					(unit 1)
 				)
@@
 		(dnp no)
 		(fields_autoplaced yes)
-		(property "Reference" "CONN_DOUT_P2"
+		(property "Reference" "C_DOUT_P2"
 			(at 107.95 63.4999 90)
 			(effects
@@
 			(project "v1"
 				(path "/c9a089ab-5af5-42df-87be-f1df643a1407/c1fbf66d-2c5c-4121-915f-86bdae7245e0"
-					(reference "CONN_DOUT_P2")
-					(unit 1)
-				)
+					(reference "C_DOUT_P2")
+					(unit 1)
+				)
