File: pcb/v1/other.kicad_sch (KiCad schematic)
At the start: 52 parts, among them J17 Conn_02x10_Top_Bottom, K1 TIANBO-HJR-4102-L, Q17 2N7002K, Q18 2N7002K, U4_RX1 TestPoint, U4_TX1 TestPoint, U5 NCP1117-3.3_SOT223, U6 NCP1117-3.3_SOT223

Commit message: Prepared for PCB ordering
Parts:
- renumbered CONN2_BTA1 to C2_BTA1, CONN2_BTA2 to C2_BTA2, CONN2_BTB1 to C2_BTB1, CONN2_BTB2 to C2_BTB2, CONN2_GND1 to C2_GND1, CONN2_I1 to C2_I1, CONN2_I2 to C2_I2, CONN2_V5 to C2_V5
Connections:
- net AGND: now also J17.1 (Pin_1); no longer J17.2 (Pin_2)
- net GND: now also J17.2 (Pin_2); no longer J17.1 (Pin_1)
- net at S3_SCK1.1: now also J17.11 (Pin_11); no longer J17.12 (Pin_12)
- net at SWDIO1.1: now also J17.5 (Pin_5); no longer J17.6 (Pin_6)
- net at IO4.1: now also J17.16 (Pin_16); no longer J17.15 (Pin_15)
- net at SWCLK1.1: now also J17.7 (Pin_7); no longer J17.8 (Pin_8)
- net at S3_MISO1.1: now also J17.9 (Pin_9); no longer J17.10 (Pin_10)
- net at J17.13 (Pin_13): now also S3_MOSI1.1
- net at J17.14 (Pin_14): no longer S3_MOSI1.1
- net at U4_RX1.1: now also J17.15 (Pin_15); no longer J17.16 (Pin_16)
- net at J17.17 (Pin_17): now also U4_TX1.1; no longer IO3.1
- net at J17.18 (Pin_18): now also IO3.1; no longer U4_TX1.1
- net at J17.19 (Pin_19): now also IO2.1; no longer IO1.1
- net at J17.20 (Pin_20): now also IO1.1; no longer IO2.1
- net at NRST1.1: now also J17.6 (Pin_6); no longer J17.5 (Pin_5)
Other:
- moved on the sheet: IO1, IO2, IO3, IO4, NRST1, SWDIO1, U4_RX1, U4_TX1
