File: pcb/v1/spare.kicad_sch (KiCad schematic)
At the start: 70 parts, among them Q11 2N7002K, Q19 2N7002K, Q20 2N7002K, Q21 2N7002K, Q22 2N7002K, Q23 2N7002K, Q24 2N7002K, Q25 2N7002K, Q26 2N7002K, Q27 2N7002K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

Commit message: Prepared for PCB ordering
Parts:
- added Q28, Q29, Q30, Q31, Q32, Q33, Q34, Q35, Q36, Q37, Q38, Q39, Q40: 2N7002K, Package_TO_SOT_SMD:SOT-23_Handsoldering, symbol Transistor_FET:2N7002K
- added RV19, RV20, RV21: R_Potentiometer, Potentiometer_SMD:Potentiometer_Bourns_TC33X_Vertical, symbol Device:R_Potentiometer
- added SPARE44, SPARE45, SPARE49: TestPoint, TestPoint:TestPoint_Pad_D2.0mm, symbol Connector:TestPoint
- added SPARE46, SPARE47, SPARE48: TestPoint, TestPoint:TestPoint_Pad_2.0x2.0mm, symbol Connector:TestPoint
- added SPARE50, SPARE51, SPARE52, SPARE53, SPARE54, SPARE55, SPARE56, SPARE57, SPARE58: TestPoint, TestPoint:TestPoint_Pad_1.5x1.5mm, symbol Connector:TestPoint
Connections:
- new net: RV21.3, SPARE57.1
- new net: SPARE45.1, SPARE47.1
- new net: RV19.2, SPARE51.1
- new net: RV19.3, SPARE52.1
- new net: RV21.1, SPARE56.1
- new net: RV20.3, SPARE54.1
- new net: RV21.2, SPARE58.1
- new net: SPARE44.1, SPARE46.1
- new net: RV20.1, SPARE53.1
- new net: RV20.2, SPARE55.1
- new net: RV19.1, SPARE50.1
- new net: SPARE48.1, SPARE49.1
