File: pcb/v1/v1.kicad_pcb (KiCad board)
At the start: 2 copper layers, 258 parts, among them J1 R_Small, J10 R_Small, J11 R_Small, J12 R_Small, J13 R_Small, J14 R_Small, J15 R_Small, J16 R_Small, J17 Conn_02x10_Top_Bottom, J2 R_Small, J3 R_Small, J4 R_Small, J5 R_Small, J6 R_Small, J7 R_Small, J8 R_Small, J9 R_Small, K1 TIANBO-HJR-4102-L, Q1 2N7002K, Q10 2N7002K, Q12 35N06, Q13 35N06, Q14 2N7002K, Q15 2N7002K, Q16 2N7002K, Q17 2N7002K, Q18 2N7002K, Q2 2N7002K, Q3 2N7002K, Q4 2N7002K, Q5 2N7002K, Q6 35N06, Q7 2N7002K, Q8 2N7002K, Q9 2N7002K, U1 MCP602, U2 MCP602, U3 MCP602, U4 MCP602, U4_RX1 TestPoint, U4_TX1 TestPoint, U5 NCP1117-3.3_SOT223, U6 NCP1117-3.3_SOT223

Commit message: Added some spare unused parts and placeholders for future design
Parts:
- added ?: , , F.Cu at (170.8, 112.5)
- added ?: , , F.Cu at (166.4, 106.0)
- added ?: , , F.Cu at (109.2, 62.9)
- added ?: , , F.Cu at (127.0, 55.0)
- added ?: , , F.Cu at (111.1, 62.9)
- added ?: , , F.Cu at (170.8, 72.4)
- added ?: , , F.Cu at (109.2, 64.7)
- added ?: , , F.Cu at (168.9, 114.3)
- added ?: , , F.Cu at (155.6, 100.4)
- added ?: , , F.Cu at (111.1, 59.1)
- added ?: , , F.Cu at (125.1, 55.0)
- added ?: , , F.Cu at (164.5, 106.0)
- added ?: , , F.Cu at (111.1, 64.7)
- added ?: , , F.Cu at (167.0, 114.3)
- added ?: , , F.Cu at (157.5, 100.4)
- added ?: , , F.Cu at (154.9, 104.2)
- added ?: , , F.Cu at (158.8, 104.2)
- added ?: , , F.Cu at (166.4, 104.2)
- added ?: , , F.Cu at (127.0, 56.8)
- added ?: , , F.Cu at (170.8, 68.6)
- added ?: , , F.Cu at (170.8, 71.1)
- added ?: , , F.Cu at (162.6, 104.2)
- added ?: , , F.Cu at (156.8, 106.0)
- added ?: , , F.Cu at (170.8, 74.9)
- added ?: , , F.Cu at (154.9, 106.0)
- added ?: , , F.Cu at (125.1, 56.8)
- added ?: , , F.Cu at (167.0, 112.5)
- added ?: , , F.Cu at (111.1, 60.9)
- added ?: , , F.Cu at (170.8, 69.8)
- added ?: , , F.Cu at (156.8, 104.2)
- added ?: , , F.Cu at (158.8, 106.0)
- added ?: , , F.Cu at (159.4, 102.2)
- added ?: , , F.Cu at (157.5, 102.2)
- added ?: , , F.Cu at (168.9, 112.5)
- added ?: , , F.Cu at (155.6, 102.2)
- added ?: , , F.Cu at (164.5, 104.2)
- added ?: , , F.Cu at (170.8, 114.3)
- added ?: , , F.Cu at (170.8, 73.7)
- added ?: , , F.Cu at (159.4, 100.4)
- added ?: , , F.Cu at (162.6, 106.0)
- added C35: 0.1, Capacitor_SMD:C_1206_3216Metric, F.Cu at (161.7, 63.5)
- added C36: 0.1, Capacitor_SMD:C_1206_3216Metric, F.Cu at (125.5, 54.0)
- added C37: 0.1, Capacitor_SMD:C_1206_3216Metric, F.Cu at (125.5, 62.2)
- added C38: 0.1, Capacitor_SMD:C_1206_3216Metric, F.Cu at (181.6, 89.7)
- added C39: 0.1, Capacitor_SMD:C_1206_3216Metric, F.Cu at (182.3, 101.4)
- added D13: LED_Dual_AAKK, Package_TO_SOT_SMD:SOT-143, F.Cu at (146.7, 75.2)
- added D14: LED_Dual_AAKK, Package_TO_SOT_SMD:SOT-143, F.Cu at (133.0, 54.3)
- added D15: LED_Dual_AAKK, Package_TO_SOT_SMD:SOT-143, F.Cu at (166.0, 59.4)
- added D16: LED_Dual_AAKK, Package_TO_SOT_SMD:SOT-143, F.Cu at (118.8, 71.2)
- added Q11: 2N7002K, Package_TO_SOT_SMD:SOT-23_Handsoldering, F.Cu at (118.1, 82.3)
- added Q19: 2N7002K, Package_TO_SOT_SMD:SOT-23_Handsoldering, F.Cu at (126.0, 82.3)
- added Q20: 2N7002K, Package_TO_SOT_SMD:SOT-23_Handsoldering, F.Cu at (131.4, 105.4)
- added Q21: 2N7002K, Package_TO_SOT_SMD:SOT-23_Handsoldering, F.Cu at (146.1, 80.9)
- added Q22: 2N7002K, Package_TO_SOT_SMD:SOT-23_Handsoldering, F.Cu at (153.0, 80.9)
- added Q23: 2N7002K, Package_TO_SOT_SMD:SOT-23_Handsoldering, F.Cu at (132.1, 59.3)
- added Q24: 2N7002K, Package_TO_SOT_SMD:SOT-23_Handsoldering, F.Cu at (123.8, 105.4)
- added Q25: 2N7002K, Package_TO_SOT_SMD:SOT-23_Handsoldering, B.Cu at (177.8, 52.7)
- added Q26: 2N7002K, Package_TO_SOT_SMD:SOT-23_Handsoldering, B.Cu at (139.7, 59.7)
- added Q27: 2N7002K, Package_TO_SOT_SMD:SOT-23_Handsoldering, F.Cu at (147.0, 105.2)
- added REF**: R_1206_3216Metric, Resistor_SMD:R_1206_3216Metric, F.Cu at (154.9, 89.3)
- added REF**: R_0805_2012Metric, Resistor_SMD:R_0805_2012Metric, F.Cu at (111.1, 79.0)
- added REF**: R_0805_2012Metric, Resistor_SMD:R_0805_2012Metric, F.Cu at (149.9, 86.0)
- added REF**: R_1206_3216Metric, Resistor_SMD:R_1206_3216Metric, F.Cu at (131.9, 68.6)
- added REF**: R_0805_2012Metric, Resistor_SMD:R_0805_2012Metric, F.Cu at (142.2, 86.0)
- added REF**: R_0805_2012Metric, Resistor_SMD:R_0805_2012Metric, F.Cu at (99.7, 71.4)
- added REF**: R_0805_2012Metric, Resistor_SMD:R_0805_2012Metric, F.Cu at (127.6, 71.5)
- added REF**: R_0805_2012Metric, Resistor_SMD:R_0805_2012Metric, F.Cu at (105.4, 75.2)
- added REF**: R_1206_3216Metric, Resistor_SMD:R_1206_3216Metric, F.Cu at (154.9, 94.2)
- added REF**: R_0805_2012Metric, Resistor_SMD:R_0805_2012Metric, F.Cu at (137.2, 56.8)
- added REF**: R_0805_2012Metric, Resistor_SMD:R_0805_2012Metric, F.Cu at (146.1, 86.0)
- added REF**: R_0805_2012Metric, Resistor_SMD:R_0805_2012Metric, F.Cu at (97.8, 67.6)
- added REF**: R_0805_2012Metric, Resistor_SMD:R_0805_2012Metric, F.Cu at (144.1, 105.1)
- added REF**: R_0805_2012Metric, Resistor_SMD:R_0805_2012Metric, F.Cu at (109.2, 75.2)
- added REF**: R_0805_2012Metric, Resistor_SMD:R_0805_2012Metric, F.Cu at (111.1, 67.6)
- added REF**: R_1206_3216Metric, Resistor_SMD:R_1206_3216Metric, F.Cu at (143.3, 108.6)
- added REF**: R_0805_2012Metric, Resistor_SMD:R_0805_2012Metric, F.Cu at (148.0, 86.0)
- added REF**: R_1206_3216Metric, Resistor_SMD:R_1206_3216Metric, F.Cu at (167.6, 94.2)
- added REF**: R_0805_2012Metric, Resistor_SMD:R_0805_2012Metric, F.Cu at (151.8, 105.7)
- added REF**: R_0805_2012Metric, Resistor_SMD:R_0805_2012Metric, F.Cu at (151.8, 86.0)
- added REF**: R_0805_2012Metric, Resistor_SMD:R_0805_2012Metric, F.Cu at (168.3, 105.1)
- added REF**: R_0805_2012Metric, Resistor_SMD:R_0805_2012Metric, F.Cu at (105.4, 79.0)
- added REF**: R_0805_2012Metric, Resistor_SMD:R_0805_2012Metric, F.Cu at (157.5, 85.4)
- added REF**: R_1206_3216Metric, Resistor_SMD:R_1206_3216Metric, F.Cu at (123.8, 93.2)
- added REF**: R_1206_3216Metric, Resistor_SMD:R_1206_3216Metric, F.Cu at (156.2, 79.8)
- added REF**: R_1206_3216Metric, Resistor_SMD:R_1206_3216Metric, F.Cu at (159.2, 108.6)
- added REF**: R_0805_2012Metric, Resistor_SMD:R_0805_2012Metric, F.Cu at (99.7, 67.6)
- added REF**: TO-252-3_TabPin2, Package_TO_SOT_SMD:TO-252-3_TabPin2, F.Cu at (116.8, 95.2)
- added REF**: R_1206_3216Metric, Resistor_SMD:R_1206_3216Metric, F.Cu at (123.8, 98.2)
- added REF**: R_1206_3216Metric, Resistor_SMD:R_1206_3216Metric, F.Cu at (160.5, 97.8)
- added REF**: R_0805_2012Metric, Resistor_SMD:R_0805_2012Metric, F.Cu at (151.8, 101.9)
- added REF**: R_0805_2012Metric, Resistor_SMD:R_0805_2012Metric, F.Cu at (129.5, 83.5)
- added REF**: R_0805_2012Metric, Resistor_SMD:R_0805_2012Metric, F.Cu at (105.4, 67.6)
- added REF**: R_0805_2012Metric, Resistor_SMD:R_0805_2012Metric, F.Cu at (149.9, 101.9)
- added REF**: R_0805_2012Metric, Resistor_SMD:R_0805_2012Metric, F.Cu at (137.2, 53.0)
- added REF**: R_1206_3216Metric, Resistor_SMD:R_1206_3216Metric, F.Cu at (134.6, 93.8)
- added REF**: R_1206_3216Metric, Resistor_SMD:R_1206_3216Metric, F.Cu at (160.0, 74.7)
- added REF**: R_1206_3216Metric, Resistor_SMD:R_1206_3216Metric, F.Cu at (174.6, 72.8)
- added REF**: R_0805_2012Metric, Resistor_SMD:R_0805_2012Metric, F.Cu at (109.2, 79.0)
- added REF**: R_0805_2012Metric, Resistor_SMD:R_0805_2012Metric, F.Cu at (129.5, 71.5)
- added REF**: R_0805_2012Metric, Resistor_SMD:R_0805_2012Metric, F.Cu at (144.1, 86.0)
- added REF**: R_1206_3216Metric, Resistor_SMD:R_1206_3216Metric, F.Cu at (179.1, 110.3)
- added REF**: R_1206_3216Metric, Resistor_SMD:R_1206_3216Metric, F.Cu at (177.2, 72.8)
- added REF**: R_1206_3216Metric, Resistor_SMD:R_1206_3216Metric, F.Cu at (164.3, 108.6)
- added REF**: R_0805_2012Metric, Resistor_SMD:R_0805_2012Metric, F.Cu at (159.4, 82.0)
- added REF**: R_0805_2012Metric, Resistor_SMD:R_0805_2012Metric, F.Cu at (105.4, 71.4)
- added REF**: R_0805_2012Metric, Resistor_SMD:R_0805_2012Metric, F.Cu at (142.2, 105.1)
- added REF**: R_1206_3216Metric, Resistor_SMD:R_1206_3216Metric, F.Cu at (167.0, 79.8)
- added REF**: R_0805_2012Metric, Resistor_SMD:R_0805_2012Metric, F.Cu at (119.4, 75.3)
- added REF**: R_1206_3216Metric, Resistor_SMD:R_1206_3216Metric, F.Cu at (160.0, 89.3)
- added REF**: R_0805_2012Metric, Resistor_SMD:R_0805_2012Metric, F.Cu at (159.4, 85.4)
- added REF**: R_1206_3216Metric, Resistor_SMD:R_1206_3216Metric, F.Cu at (157.5, 89.3)
- added REF**: R_0805_2012Metric, Resistor_SMD:R_0805_2012Metric, F.Cu at (160.7, 105.1)
- added REF**: R_0805_2012Metric, Resistor_SMD:R_0805_2012Metric, F.Cu at (155.6, 85.4)
- added REF**: R_1206_3216Metric, Resistor_SMD:R_1206_3216Metric, F.Cu at (174.6, 79.8)
- added REF**: R_0805_2012Metric, Resistor_SMD:R_0805_2012Metric, F.Cu at (121.9, 83.5)
- added REF**: R_0805_2012Metric, Resistor_SMD:R_0805_2012Metric, F.Cu at (142.2, 89.8)
- added REF**: R_1206_3216Metric, Resistor_SMD:R_1206_3216Metric, F.Cu at (155.4, 97.8)
- added REF**: R_1206_3216Metric, Resistor_SMD:R_1206_3216Metric, F.Cu at (157.5, 74.7)
- added REF**: R_1206_3216Metric, Resistor_SMD:R_1206_3216Metric, F.Cu at (165.1, 89.3)
- added REF**: R_0805_2012Metric, Resistor_SMD:R_0805_2012Metric, F.Cu at (99.7, 75.2)
- added REF**: R_1206_3216Metric, Resistor_SMD:R_1206_3216Metric, F.Cu at (122.6, 110.5)
- added REF**: R_0805_2012Metric, Resistor_SMD:R_0805_2012Metric, F.Cu at (171.4, 84.7)
- added REF**: R_1206_3216Metric, Resistor_SMD:R_1206_3216Metric, F.Cu at (169.4, 108.6)
- added REF**: TestPoint_Keystone_5019_Miniature, TestPoint:TestPoint_Keystone_5019_Miniature, B.Cu at (179.7, 86.4)
- added REF**: R_0805_2012Metric, Resistor_SMD:R_0805_2012Metric, B.Cu at (149.2, 61.0)
- added REF**: R_1206_3216Metric, Resistor_SMD:R_1206_3216Metric, B.Cu at (131.2, 115.4)
- added REF**: R_1206_3216Metric, Resistor_SMD:R_1206_3216Metric, F.Cu at (182.2, 72.8)
- added REF**: R_0805_2012Metric, Resistor_SMD:R_0805_2012Metric, B.Cu at (156.2, 61.0)
- added REF**: R_1206_3216Metric, Resistor_SMD:R_1206_3216Metric, B.Cu at (141.4, 115.4)
- added REF**: R_1206_3216Metric, Resistor_SMD:R_1206_3216Metric, B.Cu at (154.7, 50.6)
- added REF**: R_1206_3216Metric, Resistor_SMD:R_1206_3216Metric, B.Cu at (115.3, 115.4)
- added REF**: R_0805_2012Metric, Resistor_SMD:R_0805_2012Metric, B.Cu at (165.1, 50.2)
- added REF**: R_1206_3216Metric, Resistor_SMD:R_1206_3216Metric, B.Cu at (126.1, 115.4)
- added REF**: TestPoint_Keystone_5019_Miniature, TestPoint:TestPoint_Keystone_5019_Miniature, B.Cu at (170.8, 78.7)
- added REF**: R_0805_2012Metric, Resistor_SMD:R_0805_2012Metric, B.Cu at (163.8, 69.8)
- added REF**: R_0805_2012Metric, Resistor_SMD:R_0805_2012Metric, B.Cu at (179.1, 94.0)
- added REF**: R_0805_2012Metric, Resistor_SMD:R_0805_2012Metric, B.Cu at (163.2, 55.2)
- added REF**: R_0805_2012Metric, Resistor_SMD:R_0805_2012Metric, F.Cu at (131.4, 65.1)
- added REF**: R_1206_3216Metric, Resistor_SMD:R_1206_3216Metric, B.Cu at (133.7, 115.4)
- added REF**: TestPoint_Keystone_5019_Miniature, TestPoint:TestPoint_Keystone_5019_Miniature, B.Cu at (179.7, 68.6)
- added REF**: R_0805_2012Metric, Resistor_SMD:R_0805_2012Metric, B.Cu at (154.3, 65.4)
- added REF**: R_0805_2012Metric, Resistor_SMD:R_0805_2012Metric, B.Cu at (161.9, 61.0)
- added REF**: R_1206_3216Metric, Resistor_SMD:R_1206_3216Metric, B.Cu at (157.9, 115.4)
- added REF**: TestPoint_Keystone_5019_Miniature, TestPoint:TestPoint_Keystone_5019_Miniature, B.Cu at (170.8, 76.2)
- added REF**: R_1206_3216Metric, Resistor_SMD:R_1206_3216Metric, B.Cu at (107.1, 68.8)
- added REF**: R_0805_2012Metric, Resistor_SMD:R_0805_2012Metric, B.Cu at (165.1, 55.2)
- added REF**: R_1206_3216Metric, Resistor_SMD:R_1206_3216Metric, B.Cu at (137.4, 120.4)
- added REF**: TestPoint_Keystone_5019_Miniature, TestPoint:TestPoint_Keystone_5019_Miniature, B.Cu at (179.7, 85.1)
- added REF**: R_1206_3216Metric, Resistor_SMD:R_1206_3216Metric, F.Cu at (172.1, 79.8)
- added REF**: R_1206_3216Metric, Resistor_SMD:R_1206_3216Metric, B.Cu at (142.0, 55.7)
- added REF**: R_0805_2012Metric, Resistor_SMD:R_0805_2012Metric, B.Cu at (115.6, 55.9)
- added REF**: TestPoint_Keystone_5019_Miniature, TestPoint:TestPoint_Keystone_5019_Miniature, B.Cu at (179.7, 90.2)
- added REF**: R_1206_3216Metric, Resistor_SMD:R_1206_3216Metric, B.Cu at (144.5, 50.6)
- added REF**: R_0805_2012Metric, Resistor_SMD:R_0805_2012Metric, B.Cu at (121.3, 52.1)
- added REF**: R_0805_2012Metric, Resistor_SMD:R_0805_2012Metric, B.Cu at (121.3, 59.7)
- added REF**: TestPoint_Keystone_5019_Miniature, TestPoint:TestPoint_Keystone_5019_Miniature, B.Cu at (170.8, 82.5)
- added REF**: R_0805_2012Metric, Resistor_SMD:R_0805_2012Metric, B.Cu at (156.2, 65.4)
- added REF**: TestPoint_Keystone_5019_Miniature, TestPoint:TestPoint_Keystone_5019_Miniature, B.Cu at (179.7, 77.5)
- added REF**: TestPoint_Keystone_5019_Miniature, TestPoint:TestPoint_Keystone_5019_Miniature, B.Cu at (179.7, 81.3)
- added REF**: R_1206_3216Metric, Resistor_SMD:R_1206_3216Metric, F.Cu at (142.2, 79.8)
- added REF**: R_0805_2012Metric, Resistor_SMD:R_0805_2012Metric, B.Cu at (123.2, 52.1)
- added REF**: R_0805_2012Metric, Resistor_SMD:R_0805_2012Metric, B.Cu at (125.1, 59.7)
- added REF**: R_0805_2012Metric, Resistor_SMD:R_0805_2012Metric, B.Cu at (151.1, 61.0)
- added REF**: R_1206_3216Metric, Resistor_SMD:R_1206_3216Metric, B.Cu at (147.1, 55.7)
- added REF**: TestPoint_Keystone_5019_Miniature, TestPoint:TestPoint_Keystone_5019_Miniature, B.Cu at (179.7, 76.2)
- added REF**: R_1206_3216Metric, Resistor_SMD:R_1206_3216Metric, B.Cu at (138.8, 115.4)
- added REF**: TestPoint_Keystone_5019_Miniature, TestPoint:TestPoint_Keystone_5019_Miniature, B.Cu at (170.8, 87.6)
- added REF**: R_0805_2012Metric, Resistor_SMD:R_0805_2012Metric, B.Cu at (157.5, 50.2)
- added REF**: R_0805_2012Metric, Resistor_SMD:R_0805_2012Metric, B.Cu at (161.3, 55.2)
- added REF**: R_0805_2012Metric, Resistor_SMD:R_0805_2012Metric, B.Cu at (117.5, 55.9)
- added REF**: R_0805_2012Metric, Resistor_SMD:R_0805_2012Metric, F.Cu at (103.5, 75.2)
- added REF**: R_0805_2012Metric, Resistor_SMD:R_0805_2012Metric, F.Cu at (107.3, 67.6)
- added REF**: TestPoint_Keystone_5019_Miniature, TestPoint:TestPoint_Keystone_5019_Miniature, B.Cu at (179.7, 83.8)
- added REF**: R_1206_3216Metric, Resistor_SMD:R_1206_3216Metric, B.Cu at (149.6, 55.7)
- added REF**: TO-252-3_TabPin2, Package_TO_SOT_SMD:TO-252-3_TabPin2, B.Cu at (170.2, 60.3)
- added REF**: R_1206_3216Metric, Resistor_SMD:R_1206_3216Metric, B.Cu at (128.7, 115.4)
- added REF**: TestPoint_Keystone_5019_Miniature, TestPoint:TestPoint_Keystone_5019_Miniature, B.Cu at (179.7, 80.0)
- added REF**: R_0805_2012Metric, Resistor_SMD:R_0805_2012Metric, B.Cu at (157.5, 55.2)
- added REF**: R_0805_2012Metric, Resistor_SMD:R_0805_2012Metric, B.Cu at (159.4, 55.2)
- added REF**: R_1206_3216Metric, Resistor_SMD:R_1206_3216Metric, B.Cu at (157.9, 121.1)
- added REF**: R_1206_3216Metric, Resistor_SMD:R_1206_3216Metric, B.Cu at (152.1, 50.6)
- added REF**: TestPoint_Keystone_5019_Miniature, TestPoint:TestPoint_Keystone_5019_Miniature, B.Cu at (179.7, 88.9)
- added REF**: R_1206_3216Metric, Resistor_SMD:R_1206_3216Metric, F.Cu at (169.5, 72.8)
- added REF**: R_0805_2012Metric, Resistor_SMD:R_0805_2012Metric, B.Cu at (121.3, 55.9)
- added REF**: R_0805_2012Metric, Resistor_SMD:R_0805_2012Metric, B.Cu at (123.2, 55.9)
- added REF**: R_0805_2012Metric, Resistor_SMD:R_0805_2012Metric, B.Cu at (154.3, 61.0)
- added REF**: R_0805_2012Metric, Resistor_SMD:R_0805_2012Metric, B.Cu at (175.9, 97.2)
- added REF**: R_1206_3216Metric, Resistor_SMD:R_1206_3216Metric, B.Cu at (152.1, 55.7)
- added REF**: R_0805_2012Metric, Resistor_SMD:R_0805_2012Metric, B.Cu at (101.0, 69.8)
- added REF**: TestPoint_Keystone_5019_Miniature, TestPoint:TestPoint_Keystone_5019_Miniature, B.Cu at (170.8, 90.2)
- added REF**: R_1206_3216Metric, Resistor_SMD:R_1206_3216Metric, B.Cu at (147.1, 50.6)
- added REF**: TestPoint_Keystone_5019_Miniature, TestPoint:TestPoint_Keystone_5019_Miniature, B.Cu at (170.8, 83.8)
- added REF**: R_0805_2012Metric, Resistor_SMD:R_0805_2012Metric, B.Cu at (123.8, 48.9)
- added REF**: R_0805_2012Metric, Resistor_SMD:R_0805_2012Metric, F.Cu at (161.3, 101.3)
- added REF**: TestPoint_Keystone_5019_Miniature, TestPoint:TestPoint_Keystone_5019_Miniature, B.Cu at (170.8, 80.0)
- added REF**: R_0805_2012Metric, Resistor_SMD:R_0805_2012Metric, B.Cu at (181.0, 94.0)
- added REF**: R_0805_2012Metric, Resistor_SMD:R_0805_2012Metric, B.Cu at (119.4, 55.9)
- added REF**: R_0805_2012Metric, Resistor_SMD:R_0805_2012Metric, B.Cu at (179.7, 97.2)
- added REF**: R_0805_2012Metric, Resistor_SMD:R_0805_2012Metric, B.Cu at (159.4, 50.2)
- added REF**: TestPoint_Keystone_5019_Miniature, TestPoint:TestPoint_Keystone_5019_Miniature, B.Cu at (170.8, 88.9)
- added REF**: R_1206_3216Metric, Resistor_SMD:R_1206_3216Metric, B.Cu at (149.6, 50.6)
- added REF**: R_0805_2012Metric, Resistor_SMD:R_0805_2012Metric, B.Cu at (99.1, 66.0)
- added REF**: R_1206_3216Metric, Resistor_SMD:R_1206_3216Metric, B.Cu at (154.7, 121.1)
- added REF**: R_0805_2012Metric, Resistor_SMD:R_0805_2012Metric, B.Cu at (173.4, 94.0)
- added REF**: R_1206_3216Metric, Resistor_SMD:R_1206_3216Metric, F.Cu at (134.6, 98.9)
- added REF**: R_0805_2012Metric, Resistor_SMD:R_0805_2012Metric, B.Cu at (158.1, 61.0)
- added REF**: R_0805_2012Metric, Resistor_SMD:R_0805_2012Metric, B.Cu at (99.1, 73.7)
- added REF**: R_0805_2012Metric, Resistor_SMD:R_0805_2012Metric, B.Cu at (99.1, 69.8)
- added REF**: R_0805_2012Metric, Resistor_SMD:R_0805_2012Metric, B.Cu at (127.6, 48.9)
- added REF**: R_0805_2012Metric, Resistor_SMD:R_0805_2012Metric, B.Cu at (117.5, 59.7)
- added REF**: R_0805_2012Metric, Resistor_SMD:R_0805_2012Metric, B.Cu at (160.0, 69.8)
- added REF**: TestPoint_Keystone_5019_Miniature, TestPoint:TestPoint_Keystone_5019_Miniature, B.Cu at (179.7, 78.7)
- added REF**: R_0805_2012Metric, Resistor_SMD:R_0805_2012Metric, B.Cu at (161.9, 65.4)
- added REF**: TestPoint_Keystone_5019_Miniature, TestPoint:TestPoint_Keystone_5019_Miniature, B.Cu at (179.7, 73.7)
- added REF**: R_0805_2012Metric, Resistor_SMD:R_0805_2012Metric, F.Cu at (125.7, 75.3)
- added REF**: TestPoint_Keystone_5019_Miniature, TestPoint:TestPoint_Keystone_5019_Miniature, B.Cu at (170.8, 77.5)
- added REF**: R_0805_2012Metric, Resistor_SMD:R_0805_2012Metric, B.Cu at (158.1, 65.4)
- added REF**: R_0805_2012Metric, Resistor_SMD:R_0805_2012Metric, B.Cu at (117.5, 52.1)
- added REF**: R_0805_2012Metric, Resistor_SMD:R_0805_2012Metric, B.Cu at (101.0, 66.0)
- added REF**: R_0805_2012Metric, Resistor_SMD:R_0805_2012Metric, B.Cu at (145.4, 61.0)
- added REF**: R_0805_2012Metric, Resistor_SMD:R_0805_2012Metric, B.Cu at (123.2, 59.7)
- added REF**: R_0805_2012Metric, Resistor_SMD:R_0805_2012Metric, B.Cu at (147.3, 61.0)
- added REF**: TestPoint_Keystone_5019_Miniature, TestPoint:TestPoint_Keystone_5019_Miniature, B.Cu at (170.8, 85.1)
- added REF**: R_0805_2012Metric, Resistor_SMD:R_0805_2012Metric, B.Cu at (161.3, 50.2)
- added REF**: R_0805_2012Metric, Resistor_SMD:R_0805_2012Metric, B.Cu at (143.5, 61.0)
- added REF**: R_1206_3216Metric, Resistor_SMD:R_1206_3216Metric, F.Cu at (179.7, 79.8)
- added REF**: R_0805_2012Metric, Resistor_SMD:R_0805_2012Metric, B.Cu at (128.9, 52.1)
- added REF**: R_1206_3216Metric, Resistor_SMD:R_1206_3216Metric, B.Cu at (142.0, 50.6)
- added REF**: R_1206_3216Metric, Resistor_SMD:R_1206_3216Metric, B.Cu at (112.2, 68.8)
- added REF**: R_0805_2012Metric, Resistor_SMD:R_0805_2012Metric, B.Cu at (177.2, 94.0)
- added REF**: R_0805_2012Metric, Resistor_SMD:R_0805_2012Metric, B.Cu at (115.6, 59.7)
- added REF**: TestPoint_Keystone_5019_Miniature, TestPoint:TestPoint_Keystone_5019_Miniature, B.Cu at (179.7, 69.8)
- added REF**: TestPoint_Keystone_5019_Miniature, TestPoint:TestPoint_Keystone_5019_Miniature, B.Cu at (179.7, 74.9)
- added REF**: R_0805_2012Metric, Resistor_SMD:R_0805_2012Metric, B.Cu at (161.9, 69.8)
- added REF**: TestPoint_Keystone_5019_Miniature, TestPoint:TestPoint_Keystone_5019_Miniature, B.Cu at (179.7, 87.6)
- added REF**: R_1206_3216Metric, Resistor_SMD:R_1206_3216Metric, B.Cu at (144.5, 55.7)
- added REF**: R_0805_2012Metric, Resistor_SMD:R_0805_2012Metric, F.Cu at (121.9, 88.0)
- added REF**: R_0805_2012Metric, Resistor_SMD:R_0805_2012Metric, B.Cu at (101.0, 73.7)
- added REF**: R_1206_3216Metric, Resistor_SMD:R_1206_3216Metric, B.Cu at (154.7, 115.4)
- added REF**: R_0805_2012Metric, Resistor_SMD:R_0805_2012Metric, B.Cu at (127.0, 52.1)
- added REF**: R_1206_3216Metric, Resistor_SMD:R_1206_3216Metric, B.Cu at (154.7, 55.7)
- added REF**: R_0805_2012Metric, Resistor_SMD:R_0805_2012Metric, B.Cu at (160.0, 65.4)
- added REF**: R_1206_3216Metric, Resistor_SMD:R_1206_3216Metric, B.Cu at (143.1, 120.4)
- added REF**: R_0805_2012Metric, Resistor_SMD:R_0805_2012Metric, B.Cu at (115.6, 52.1)
- added REF**: R_0805_2012Metric, Resistor_SMD:R_0805_2012Metric, B.Cu at (119.4, 52.1)
- added REF**: R_1206_3216Metric, Resistor_SMD:R_1206_3216Metric, B.Cu at (117.3, 68.8)
- added REF**: TestPoint_Keystone_5019_Miniature, TestPoint:TestPoint_Keystone_5019_Miniature, B.Cu at (179.7, 82.5)
- added REF**: R_1206_3216Metric, Resistor_SMD:R_1206_3216Metric, F.Cu at (182.2, 79.8)
- added REF**: TestPoint_Keystone_5019_Miniature, TestPoint:TestPoint_Keystone_5019_Miniature, B.Cu at (179.7, 71.1)
- added REF**: TestPoint_Keystone_5019_Miniature, TestPoint:TestPoint_Keystone_5019_Miniature, B.Cu at (179.7, 72.4)
- added REF**: R_0805_2012Metric, Resistor_SMD:R_0805_2012Metric, B.Cu at (175.3, 94.0)
- added REF**: R_0805_2012Metric, Resistor_SMD:R_0805_2012Metric, B.Cu at (131.4, 48.9)
- added REF**: R_0805_2012Metric, Resistor_SMD:R_0805_2012Metric, B.Cu at (125.1, 52.1)
- added REF**: R_0805_2012Metric, Resistor_SMD:R_0805_2012Metric, B.Cu at (119.4, 59.7)
- added REF**: R_0805_2012Metric, Resistor_SMD:R_0805_2012Metric, B.Cu at (163.2, 50.2)
- added REF**: TestPoint_Keystone_5019_Miniature, TestPoint:TestPoint_Keystone_5019_Miniature, B.Cu at (170.8, 86.4)
- added REF**: R_0805_2012Metric, Resistor_SMD:R_0805_2012Metric, B.Cu at (160.0, 61.0)
- added REF**: TestPoint_Keystone_5019_Miniature, TestPoint:TestPoint_Keystone_5019_Miniature, B.Cu at (170.8, 81.3)
- added REF**: R_1206_3216Metric, Resistor_SMD:R_1206_3216Metric, F.Cu at (172.1, 72.8)
- added REF**: R_1206_3216Metric, Resistor_SMD:R_1206_3216Metric, B.Cu at (136.3, 115.4)
- added REF**: R_1206_3216Metric, Resistor_SMD:R_1206_3216Metric, F.Cu at (157.4, 94.2)
- added REF**: R_1206_3216Metric, Resistor_SMD:R_1206_3216Metric, F.Cu at (181.6, 115.4)
- added REF**: R_1206_3216Metric, Resistor_SMD:R_1206_3216Metric, F.Cu at (169.5, 79.8)
- added REF**: R_0805_2012Metric, Resistor_SMD:R_0805_2012Metric, F.Cu at (107.3, 79.0)
- added REF**: R_0805_2012Metric, Resistor_SMD:R_0805_2012Metric, F.Cu at (103.5, 67.6)
- added REF**: R_1206_3216Metric, Resistor_SMD:R_1206_3216Metric, F.Cu at (162.6, 89.3)
- added REF**: R_1206_3216Metric, Resistor_SMD:R_1206_3216Metric, F.Cu at (177.2, 79.8)
- added REF**: R_0805_2012Metric, Resistor_SMD:R_0805_2012Metric, F.Cu at (137.2, 60.6)
- added REF**: R_0805_2012Metric, Resistor_SMD:R_0805_2012Metric, F.Cu at (123.2, 79.7)
- added REF**: R_0805_2012Metric, Resistor_SMD:R_0805_2012Metric, F.Cu at (120.7, 79.7)
- added REF**: R_1206_3216Metric, Resistor_SMD:R_1206_3216Metric, F.Cu at (160.0, 94.2)
- added REF**: R_1206_3216Metric, Resistor_SMD:R_1206_3216Metric, F.Cu at (165.0, 94.2)
- added REF**: R_0805_2012Metric, Resistor_SMD:R_0805_2012Metric, F.Cu at (118.1, 88.0)
- added REF**: R_0805_2012Metric, Resistor_SMD:R_0805_2012Metric, F.Cu at (142.2, 101.2)
- added REF**: R_0805_2012Metric, Resistor_SMD:R_0805_2012Metric, F.Cu at (117.5, 75.3)
- added REF**: R_0805_2012Metric, Resistor_SMD:R_0805_2012Metric, F.Cu at (111.1, 71.4)
- added REF**: R_1206_3216Metric, Resistor_SMD:R_1206_3216Metric, F.Cu at (154.1, 112.4)
- added REF**: R_0805_2012Metric, Resistor_SMD:R_0805_2012Metric, F.Cu at (116.2, 88.0)
- added REF**: R_0805_2012Metric, Resistor_SMD:R_0805_2012Metric, F.Cu at (144.1, 93.6)
- added REF**: R_0805_2012Metric, Resistor_SMD:R_0805_2012Metric, F.Cu at (129.5, 75.3)
- added REF**: R_0805_2012Metric, Resistor_SMD:R_0805_2012Metric, F.Cu at (142.2, 97.4)
- added REF**: R_0805_2012Metric, Resistor_SMD:R_0805_2012Metric, F.Cu at (144.1, 89.8)
- added REF**: R_0805_2012Metric, Resistor_SMD:R_0805_2012Metric, F.Cu at (121.3, 75.3)
- added REF**: R_0805_2012Metric, Resistor_SMD:R_0805_2012Metric, F.Cu at (109.2, 67.6)
- added REF**: R_1206_3216Metric, Resistor_SMD:R_1206_3216Metric, F.Cu at (127.8, 101.0)
- added REF**: R_1206_3216Metric, Resistor_SMD:R_1206_3216Metric, F.Cu at (172.1, 93.2)
- added REF**: R_1206_3216Metric, Resistor_SMD:R_1206_3216Metric, F.Cu at (134.6, 103.9)
- added REF**: R_1206_3216Metric, Resistor_SMD:R_1206_3216Metric, F.Cu at (181.6, 110.3)
- added REF**: R_0805_2012Metric, Resistor_SMD:R_0805_2012Metric, F.Cu at (123.8, 75.3)
- added REF**: R_0805_2012Metric, Resistor_SMD:R_0805_2012Metric, F.Cu at (97.8, 75.2)
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Routing:
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
Commit message: Prepared for PCB ordering
Parts:
- removed the ? at (166.4, 106.0)
- removed the ? at (170.8, 72.4)
- removed the ? at (109.2, 64.7)
- removed the ? at (155.6, 100.4)
- removed the ? at (164.5, 106.0)
- removed the ? at (111.1, 64.7)
- removed the ? at (166.4, 104.2)
- removed the ? at (170.8, 68.6)
- removed the ? at (170.8, 71.1)
- removed the ? at (162.6, 104.2)
- removed the ? at (170.8, 74.9)
- removed the ? at (170.8, 69.8)
- removed the ? at (155.6, 102.2)
- removed the ? at (164.5, 104.2)
- removed the ? at (170.8, 73.7)
- removed the ? at (162.6, 106.0)
- removed the REF** at (154.9, 89.3)
- removed the REF** at (99.7, 71.4)
- removed the REF** at (105.4, 75.2)
- removed the REF** at (111.1, 67.6)
- removed the REF** at (168.3, 105.1)
- removed the REF** at (157.5, 85.4)
- removed the REF** at (99.7, 67.6)
- removed the REF** at (151.8, 101.9)
- removed the REF** at (129.5, 83.5)
- removed the REF** at (105.4, 67.6)
- removed the REF** at (137.2, 53.0)
- removed the REF** at (159.4, 82.0)
- removed the REF** at (105.4, 71.4)
- removed the REF** at (119.4, 75.3)
- removed the REF** at (160.0, 89.3)
- removed the REF** at (159.4, 85.4)
- removed the REF** at (157.5, 89.3)
- removed the REF** at (160.7, 105.1)
- removed the REF** at (155.6, 85.4)
- removed the REF** at (142.2, 89.8)
- removed the REF** at (165.1, 89.3)
- removed the REF** at (99.7, 75.2)
- removed the REF** at (179.7, 86.4)
- removed the REF** at (165.1, 50.2)
- removed the REF** at (126.1, 115.4)
- removed the REF** at (170.8, 78.7)
- removed the REF** at (179.7, 68.6)
- removed the REF** at (157.9, 115.4)
- removed the REF** at (170.8, 76.2)
- removed the REF** at (179.7, 85.1)
- removed the REF** at (115.6, 55.9)
- removed the REF** at (179.7, 90.2)
- removed the REF** at (170.8, 82.5)
- removed the REF** at (179.7, 77.5)
- removed the REF** at (179.7, 81.3)
- removed the REF** at (147.1, 55.7)
- removed the REF** at (179.7, 76.2)
- removed the REF** at (138.8, 115.4)
- removed the REF** at (170.8, 87.6)
- removed the REF** at (157.5, 50.2)
- removed the REF** at (103.5, 75.2)
- removed the REF** at (179.7, 83.8)
- removed the REF** at (149.6, 55.7)
- removed the REF** at (179.7, 80.0)
- removed the REF** at (157.9, 121.1)
- removed the REF** at (179.7, 88.9)
- removed the REF** at (152.1, 55.7)
- removed the REF** at (170.8, 90.2)
- removed the REF** at (170.8, 83.8)
- removed the REF** at (161.3, 101.3)
- removed the REF** at (170.8, 80.0)
- removed the REF** at (170.8, 88.9)
- removed the REF** at (154.7, 121.1)
- removed the REF** at (173.4, 94.0)
- removed the REF** at (117.5, 59.7)
- removed the REF** at (179.7, 78.7)
- removed the REF** at (179.7, 73.7)
- removed the REF** at (170.8, 77.5)
- removed the REF** at (170.8, 85.1)
- removed the REF** at (115.6, 59.7)
- removed the REF** at (179.7, 69.8)
- removed the REF** at (179.7, 74.9)
- removed the REF** at (179.7, 87.6)
- removed the REF** at (144.5, 55.7)
- removed the REF** at (154.7, 115.4)
- removed the REF** at (179.7, 82.5)
- removed the REF** at (179.7, 71.1)
- removed the REF** at (179.7, 72.4)
- removed the REF** at (163.2, 50.2)
- removed the REF** at (170.8, 86.4)
- removed the REF** at (170.8, 81.3)
- removed the REF** at (136.3, 115.4)
- removed the REF** at (157.4, 94.2)
- removed the REF** at (103.5, 67.6)
- removed the REF** at (162.6, 89.3)
- removed the REF** at (137.2, 60.6)
- removed the REF** at (160.0, 94.2)
- removed the REF** at (111.1, 71.4)
- removed the REF** at (144.1, 93.6)
- removed the REF** at (129.5, 75.3)
- removed the REF** at (142.2, 97.4)
- removed the REF** at (144.1, 89.8)
- removed the REF** at (109.2, 67.6)
- removed the REF** at (114.9, 83.5)
- removed the REF** at (163.2, 85.4)
- removed the REF** at (133.3, 83.0)
- removed the REF** at (101.6, 71.4)
- removed the REF** at (142.2, 93.6)
- removed the REF** at (101.6, 67.6)
- removed the REF** at (161.3, 85.4)
- removed the REF** at (167.6, 89.3)
- removed the REF** at (144.1, 97.4)
- removed the REF** at (134.6, 88.7)
- removed the REF** at (139.1, 53.0)
- removed the REF** at (103.5, 71.4)
- removed the REF** at (127.6, 75.3)
- removed the REF** at (109.2, 71.4)
- removed the REF** at (101.6, 75.2)
- added ?: , , F.Cu at (160.5, 89.0)
- added ?: , , F.Cu at (160.5, 90.8)
- added ?: , , F.Cu at (162.8, 89.0)
- added ?: , , F.Cu at (159.1, 81.5)
- added ?: , , F.Cu at (159.1, 83.3)
- added ?: , , F.Cu at (163.7, 86.2)
- added ?: , , F.Cu at (154.7, 89.0)
- added ?: , , F.Cu at (154.7, 90.8)
- added ?: , , F.Cu at (163.7, 84.4)
- added ?: , , F.Cu at (162.8, 90.8)
- added ?: , , F.Cu at (157.0, 90.8)
- added ?: , , F.Cu at (157.0, 89.0)
- added J18: R_Small, Resistor_SMD:R_1206_3216Metric_Pad1.30x1.75mm_HandSolder, F.Cu at (118.5, 126.6)
- added J19: R_Small, Resistor_SMD:R_1206_3216Metric_Pad1.30x1.75mm_HandSolder, F.Cu at (142.2, 125.9)
- added J20: R_Small, Resistor_SMD:R_1206_3216Metric_Pad1.30x1.75mm_HandSolder, F.Cu at (166.1, 124.9)
- added Q28: 2N7002K, Package_TO_SOT_SMD:SOT-23_Handsoldering, B.Cu at (175.3, 51.4)
- added Q29: 2N7002K, Package_TO_SOT_SMD:SOT-23_Handsoldering, B.Cu at (181.6, 57.8)
- added Q30: 2N7002K, Package_TO_SOT_SMD:SOT-23_Handsoldering, F.Cu at (157.2, 85.5)
- added Q31: 2N7002K, Package_TO_SOT_SMD:SOT-23_Handsoldering, F.Cu at (161.1, 85.5)
- added Q32: 2N7002K, Package_TO_SOT_SMD:SOT-23_Handsoldering, F.Cu at (158.8, 93.4)
- added Q33: 2N7002K, Package_TO_SOT_SMD:SOT-23_Handsoldering, F.Cu at (165.4, 88.4)
- added Q34: 2N7002K, Package_TO_SOT_SMD:SOT-23_Handsoldering, B.Cu at (146.7, 56.1)
- added Q35: 2N7002K, Package_TO_SOT_SMD:SOT-23_Handsoldering, B.Cu at (151.1, 56.2)
- added Q36: 2N7002K, Package_TO_SOT_SMD:SOT-23_Handsoldering, B.Cu at (114.6, 58.6)
- added Q37: 2N7002K, Package_TO_SOT_SMD:SOT-23_Handsoldering, B.Cu at (156.1, 116.4)
- added Q38: 2N7002K, Package_TO_SOT_SMD:SOT-23_Handsoldering, B.Cu at (156.0, 121.9)
- added Q39: 2N7002K, Package_TO_SOT_SMD:SOT-23_Handsoldering, B.Cu at (137.3, 116.3)
- added Q40: 2N7002K, Package_TO_SOT_SMD:SOT-23_Handsoldering, B.Cu at (124.8, 115.8)
- added REF**: R_1206_3216Metric, Resistor_SMD:R_1206_3216Metric, F.Cu at (111.1, 88.5)
- added REF**: R_1206_3216Metric, Resistor_SMD:R_1206_3216Metric, F.Cu at (122.4, 65.4)
- added REF**: R_0805_2012Metric, Resistor_SMD:R_0805_2012Metric, B.Cu at (178.6, 68.8)
- added REF**: R_0805_2012Metric, Resistor_SMD:R_0805_2012Metric, B.Cu at (158.8, 114.9)
- added REF**: R_1206_3216Metric, Resistor_SMD:R_1206_3216Metric, F.Cu at (129.2, 77.6)
- added REF**: TestPoint_Pad_2.0x2.0mm, TestPoint:TestPoint_Pad_2.0x2.0mm, B.Cu at (158.8, 104.1)
- added REF**: TestPoint_Pad_2.0x2.0mm, TestPoint:TestPoint_Pad_2.0x2.0mm, B.Cu at (132.1, 110.5)
- added REF**: R_0805_2012Metric, Resistor_SMD:R_0805_2012Metric, B.Cu at (174.8, 68.8)
- added REF**: TestPoint_Pad_2.0x2.0mm, TestPoint:TestPoint_Pad_2.0x2.0mm, B.Cu at (158.8, 88.9)
- added REF**: TestPoint_Pad_2.0x2.0mm, TestPoint:TestPoint_Pad_2.0x2.0mm, B.Cu at (134.6, 110.5)
- added REF**: R_0805_2012Metric, Resistor_SMD:R_0805_2012Metric, B.Cu at (169.2, 68.8)
- added REF**: R_0805_2012Metric, Resistor_SMD:R_0805_2012Metric, B.Cu at (176.7, 68.8)
- added REF**: R_0805_2012Metric, Resistor_SMD:R_0805_2012Metric, B.Cu at (180.5, 68.8)
- added REF**: TestPoint_Pad_2.0x2.0mm, TestPoint:TestPoint_Pad_2.0x2.0mm, B.Cu at (158.8, 94.0)
- added REF**: TestPoint_Pad_2.0x2.0mm, TestPoint:TestPoint_Pad_2.0x2.0mm, B.Cu at (127.0, 110.5)
- added REF**: R_0805_2012Metric, Resistor_SMD:R_0805_2012Metric, F.Cu at (173.2, 129.9)
- added REF**: R_0805_2012Metric, Resistor_SMD:R_0805_2012Metric, B.Cu at (153.7, 119.7)
- added REF**: R_0805_2012Metric, Resistor_SMD:R_0805_2012Metric, B.Cu at (182.4, 68.8)
- added REF**: TestPoint_Pad_2.0x2.0mm, TestPoint:TestPoint_Pad_2.0x2.0mm, B.Cu at (116.0, 110.5)
- added REF**: R_0805_2012Metric, Resistor_SMD:R_0805_2012Metric, B.Cu at (171.1, 68.8)
- added REF**: TestPoint_Pad_2.0x2.0mm, TestPoint:TestPoint_Pad_2.0x2.0mm, B.Cu at (158.8, 96.5)
- added REF**: TestPoint_Pad_2.0x2.0mm, TestPoint:TestPoint_Pad_2.0x2.0mm, B.Cu at (129.5, 110.5)
- added REF**: R_1206_3216Metric, Resistor_SMD:R_1206_3216Metric, B.Cu at (117.2, 116.6)
- added REF**: R_0805_2012Metric, Resistor_SMD:R_0805_2012Metric, B.Cu at (172.8, 68.8)
- added REF**: R_0805_2012Metric, Resistor_SMD:R_0805_2012Metric, B.Cu at (158.8, 107.3)
- added REF**: R_0805_2012Metric, Resistor_SMD:R_0805_2012Metric, B.Cu at (158.8, 111.1)
- added REF**: TestPoint_Pad_2.0x2.0mm, TestPoint:TestPoint_Pad_2.0x2.0mm, B.Cu at (158.8, 91.4)
- added REF**: R_1206_3216Metric, Resistor_SMD:R_1206_3216Metric, F.Cu at (111.1, 83.4)
- added REF**: R_1206_3216Metric, Resistor_SMD:R_1206_3216Metric, F.Cu at (149.8, 74.8)
- added REF**: R_1206_3216Metric, Resistor_SMD:R_1206_3216Metric, F.Cu at (117.4, 65.4)
- added REF**: R_0805_2012Metric, Resistor_SMD:R_0805_2012Metric, F.Cu at (175.1, 129.9)
- added REF**: SOIC-16_3.9x9.9mm_P1.27mm, Package_SO:SOIC-16_3.9x9.9mm_P1.27mm, F.Cu at (102.6, 70.9)
- added REF**: R_1206_3216Metric, Resistor_SMD:R_1206_3216Metric, F.Cu at (129.2, 82.6)
- added REF**: R_0805_2012Metric, Resistor_SMD:R_0805_2012Metric, F.Cu at (128.8, 62.3)
- added REF**: R_1206_3216Metric, Resistor_SMD:R_1206_3216Metric, F.Cu at (127.2, 65.4)
- added REF**: R_0805_2012Metric, Resistor_SMD:R_0805_2012Metric, F.Cu at (165.1, 133.8)
- added REF**: R_0805_2012Metric, Resistor_SMD:R_0805_2012Metric, F.Cu at (132.8, 86.2)
- added REF**: R_0805_2012Metric, Resistor_SMD:R_0805_2012Metric, F.Cu at (129.5, 86.2)
- added REF**: R_0805_2012Metric, Resistor_SMD:R_0805_2012Metric, F.Cu at (181.8, 132.9)
- added REF**: R_0805_2012Metric, Resistor_SMD:R_0805_2012Metric, F.Cu at (133.6, 61.0)
- added RV19: R_Potentiometer, Potentiometer_SMD:Potentiometer_Bourns_TC33X_Vertical, F.Cu at (164.8, 104.6)
- added RV20: R_Potentiometer, Potentiometer_SMD:Potentiometer_Bourns_TC33X_Vertical, F.Cu at (110.7, 68.3)
- added RV21: R_Potentiometer, Potentiometer_SMD:Potentiometer_Bourns_TC33X_Vertical, F.Cu at (143.7, 93.2)
- added SPARE44: TestPoint, TestPoint:TestPoint_Pad_D2.0mm, F.Cu at (131.7, 50.4)
- added SPARE45: TestPoint, TestPoint:TestPoint_Pad_D2.0mm, F.Cu at (128.3, 50.4)
- added SPARE46: TestPoint, TestPoint:TestPoint_Pad_2.0x2.0mm, F.Cu at (134.6, 94.7)
- added SPARE47: TestPoint, TestPoint:TestPoint_Pad_2.0x2.0mm, F.Cu at (124.6, 88.0)
- added SPARE48: TestPoint, TestPoint:TestPoint_Pad_2.0x2.0mm, B.Cu at (172.6, 93.9)
- added SPARE49: TestPoint, TestPoint:TestPoint_Pad_D2.0mm, B.Cu at (164.5, 50.0)
- added SPARE50: TestPoint, TestPoint:TestPoint_Pad_1.5x1.5mm, F.Cu at (161.1, 103.4)
- added SPARE51: TestPoint, TestPoint:TestPoint_Pad_1.5x1.5mm, F.Cu at (168.2, 104.6)
- added SPARE52: TestPoint, TestPoint:TestPoint_Pad_1.5x1.5mm, F.Cu at (161.1, 105.8)
- added SPARE53: TestPoint, TestPoint:TestPoint_Pad_1.5x1.5mm, F.Cu at (109.6, 72.1)
- added SPARE54: TestPoint, TestPoint:TestPoint_Pad_1.5x1.5mm, F.Cu at (111.9, 72.1)
- added SPARE55: TestPoint, TestPoint:TestPoint_Pad_1.5x1.5mm, F.Cu at (110.7, 64.9)
- added SPARE56: TestPoint, TestPoint:TestPoint_Pad_1.5x1.5mm, F.Cu at (142.5, 97.3)
- added SPARE57: TestPoint, TestPoint:TestPoint_Pad_1.5x1.5mm, F.Cu at (144.8, 97.3)
- added SPARE58: TestPoint, TestPoint:TestPoint_Pad_1.5x1.5mm, F.Cu at (143.6, 89.6)
- J17: moved to F.Cu
- moved REF** 26.0 mm to (108.6, 93.2)
- moved SPARE21 19.1 mm to (133.5, 79.6), turned to -90 degrees
- moved SPARE26 18.4 mm to (133.5, 84.1), turned to -90 degrees
- moved D16 17.5 mm to (132.8, 81.8), turned to -90 degrees
- moved SPARE22 16.8 mm to (131.6, 79.6), turned to -90 degrees
- moved SPARE25 16.0 mm to (131.6, 84.1), turned to -90 degrees
- moved REF** 12.0 mm to (116.1, 62.3)
- moved REF** 12.0 mm to (118.0, 62.3)
- moved REF** 12.0 mm to (119.9, 62.3)
- moved REF** 12.0 mm to (121.8, 62.3)
- moved SPARE16 8.40 mm to (139.1, 54.6), turned to 90 degrees
- moved SPARE15 6.57 mm to (137.2, 54.6), turned to 90 degrees
- moved SPARE17 6.42 mm to (139.0, 49.9), turned to 90 degrees
- moved SPARE28 6.14 mm to (128.9, 74.1)
- moved D14 5.60 mm to (138.2, 52.3), turned to 90 degrees
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- renumbered CONN2_BTA1 to C2_BTA1, CONN2_BTA2 to C2_BTA2, CONN2_BTB1 to C2_BTB1, CONN2_BTB2 to C2_BTB2, CONN2_GND1 to C2_GND1, CONN2_I1 to C2_I1, CONN2_I2 to C2_I2, CONN2_V5 to C2_V5, CONN_AIN1 to C_AIN1, CONN_AIN2 to C_AIN2, CONN_AIN3 to C_AIN3, CONN_AIN4 to C_AIN4, CONN_AIN5 to C_AIN5, CONN_AIN6 to C_AIN6, CONN_AOUT1 to C_AOUT1, CONN_AOUT2 to C_AOUT2, CONN_DIN1 to C_DIN1, CONN_DIN2 to C_DIN2, CONN_DIN3 to C_DIN3, CONN_DIN4 to C_DIN4, CONN_DIN5 to C_DIN5, CONN_DIN6 to C_DIN6, CONN_DOUT1 to C_DOUT1, CONN_DOUT2 to C_DOUT2, CONN_DOUT3 to C_DOUT3, CONN_DOUT4 to C_DOUT4, CONN_DOUT5 to C_DOUT5, CONN_DOUT_P1 to C_DOUT_P1, CONN_DOUT_P2 to C_DOUT_P2, CONN_DOUT_P3 to C_DOUT_P3, CONN_DOUT_P_GND1 to C_DOUT_P_GND1
Connections:
- C1 pad 1: A3V -> Net-(U1C-V+)
- C15 pad 1: A3V -> Net-(U4C-V+)
- C16 pad 1: A3V -> Net-(U4C-V+)
- C4 pad 1: A3V -> Net-(U1C-V+)
- C5 pad 1: A3V -> Net-(U2C-V+)
- C6 pad 1: A3V -> Net-(U2C-V+)
- IO1 pad 1: Net-(J17-Pin_19) -> Net-(J17-Pin_20)
- IO2 pad 1: Net-(J17-Pin_20) -> Net-(J17-Pin_19)
- IO3 pad 1: Net-(J17-Pin_17) -> Net-(J17-Pin_18)
- IO4 pad 1: Net-(J17-Pin_15) -> Net-(J17-Pin_16)
- J1 pad 1: A3V -> Net-(U1C-V+)
- J11 pad 1: A3V -> Net-(U4C-V+)
- J12 pad 1: A3V -> Net-(U4C-V+)
- J17 pad 1: GND -> AGND
- J17 pad 10: Net-(J17-Pin_10) -> unconnected-(J17-Pin_10-Pad10)
- J17 pad 11: unconnected-(J17-Pin_11-Pad11) -> Net-(J17-Pin_11)
- J17 pad 12: Net-(J17-Pin_12) -> unconnected-(J17-Pin_12-Pad12)
- J17 pad 13: unconnected-(J17-Pin_13-Pad13) -> Net-(J17-Pin_13)
- J17 pad 14: Net-(J17-Pin_14) -> unconnected-(J17-Pin_14-Pad14)
- J17 pad 2: AGND -> GND
- J17 pad 7: unconnected-(J17-Pin_7-Pad7) -> Net-(J17-Pin_7)
- J17 pad 8: Net-(J17-Pin_8) -> unconnected-(J17-Pin_8-Pad8)
- J17 pad 9: unconnected-(J17-Pin_9-Pad9) -> Net-(J17-Pin_9)
- J3 pad 1: A3V -> Net-(U1C-V+)
- J5 pad 1: A3V -> Net-(U2C-V+)
- J6 pad 1: A3V -> Net-(U2C-V+)
- NRST1 pad 1: Net-(J17-Pin_5) -> Net-(J17-Pin_6)
- NRST1B pad 1: Net-(J17-Pin_5) -> Net-(J17-Pin_6)
- S3_MISO1 pad 1: Net-(J17-Pin_10) -> Net-(J17-Pin_9)
- S3_MOSI1 pad 1: Net-(J17-Pin_14) -> Net-(J17-Pin_13)
- S3_SCK1 pad 1: Net-(J17-Pin_12) -> Net-(J17-Pin_11)
- SWCLK1 pad 1: Net-(J17-Pin_8) -> Net-(J17-Pin_7)
- SWDIO1 pad 1: Net-(J17-Pin_6) -> Net-(J17-Pin_5)
- U1 pad 8: A3V -> Net-(U1C-V+)
- U2 pad 8: A3V -> Net-(U2C-V+)
- U4 pad 8: A3V -> Net-(U4C-V+)
- U4_RX1 pad 1: Net-(J17-Pin_16) -> Net-(J17-Pin_15)
- U4_TX1 pad 1: Net-(J17-Pin_18) -> Net-(J17-Pin_17)
Routing:
- net A3V: track 525.3 -> 399.4 mm
- net Net-(J17-Pin_6): track 7.52 -> 118.2 mm, vias 0 -> 1
- net Net-(J17-Pin_5): track 114.1 -> 7.40 mm, vias 1 -> 0
- net (no net): track 0.00 -> 97.4 mm, vias 13 -> 19
- net Net-(SPARE45-Pad1): track 0.00 -> 50.4 mm
- net Net-(SPARE48-Pad1): track 0.00 -> 48.7 mm
- net Net-(SPARE44-Pad1): track 0.00 -> 47.0 mm
- net Net-(U4C-V+): track 0.00 -> 45.3 mm
- net Net-(U1C-V+): track 0.00 -> 38.8 mm
- net Net-(U2C-V+): track 0.00 -> 38.0 mm
- net Net-(J17-Pin_9): track 0.00 -> 13.0 mm
- net Net-(J17-Pin_10): track 13.0 -> 0.00 mm
- net Net-(J17-Pin_12): track 12.8 -> 0.00 mm
- net Net-(J17-Pin_11): track 0.00 -> 12.8 mm
- net Net-(J17-Pin_14): track 12.3 -> 0.00 mm
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Other:
- board outline added: 90.2 x 110.8 mm
- board text added: "0.5"
- board text added: "0.635"
- board text added: "3V"
- board text added: "5V"
- board text added: "???????"
- board text added: "A3V"
- board text added: "AGND"
- board text added: "B1"
- board text added: "B2"
- board text added: "GND"
- board text added: "MISO"
- board text added: "MOSI"
- board text added: "P1"
- board text added: "P2"
- board text added: "POT"
- board text added: "POT EXT"
- board text added: "RX"
- board text added: "SCK"
- board text added: "TX"
- board text added: "ctlpie v1.0 sep 2025"
- board text removed: "- Oscillaor - LAMP"
- board text removed: "Connectors/Jumpers wire ! Flashlight CONNECTOR IS ON THE WORNG SIDE !!!"
